File: BalancerREF/BalancerREF.kicad_sch (KiCad schematic)
At the start: 80 parts, among them J1 USB4105-GF-A, J2 LiPo 500mAh PROTECTED, J3 MAG+ / MAG- PTH, J4 GPS MODULE 3V3 UART, J5 OPTICAL HEAD 7-WAY, Q3 AO3401A, Q4 AO3401A, SW1 POWER, SW2 ACQUIRE, SW3 BOOT / SERVICE, SW4 RESET, U1 ESP32-S3-MINI-1-N8, U10 SN74LVC1G123DCTR, U2 IIS3DWBTR, U3 LM1815MX/NOPB, U5 MCP73831T-2ACI/OT, U6 TPS63031DSKR, U7 SRV05-4MR6T1G, U9 SN74LVC1G08DBVR

Commit message: feat: split optical head to its own board, place both PCBs
BalancerREF main board (50 x 50, 4 layer):
- optical front end removed to BalancerREF_OptHead; J5 7-way cable connector
  added, with ground interleaved between OPT_LED_EN and OPT_COMP
- SW4 (RESET) removed - SW1 feeds U6 VIN and EN, so the power slide already
  power-cycles the MCU; R4/C10/TP13 still hold EN high and probeable
- R5 removed - it duplicated R9's 10k BOOT pull-up on the same net
- all 83 footprints placed: ICs, connectors, switches and test points on the
  front, passives on the back under their own IC's power pins
- M2.5 mounting holes at the four corners
- UP / LEFT orientation markers on F.SilkS for vertical mounting with the
  ESP32 left and USB-C right
- DRC 2, both the U1 library courtyard overlapping the corner holes; U1's real
  antenna keepout is off-board thanks to the overhang

BalancerREF_OptHead (25 x 50, 2 layer), new PCB:
- every part on the front so B.Cu is an uninterrupted GND pour, which matters
  more than a clean optical face given the transimpedance summing node
- D1 centred on the optical axis, PD1 18 mm directly below, J5 on the bottom
- DRC 0

Verification:
- verify_netlist.py spec updated for the split and re-passing honestly. It had
  been reporting PASS against a stale netlist; regenerating that netlist made it
  crash, which is what the spec update fixes. PASS: 43 exact circuit nets,
  280 pin endpoints, 128 IC pads
- verify_head.py unchanged, PASS: 16 exact circuit nets, 63 pin endpoints
- review/ artifacts regenerated from the current schematic

Lens keepout radius and the D1-PD1 spacing are estimates pending the real
Ledil TINA holder dimensions.

Co-Authored-By: Claude Opus 5 (1M context) <noreply@anthropic.com>
Parts:
- removed R5: 10k, Resistor_SMD:R_0603_1608Metric, symbol Device:R
- removed SW4: RESET, Button_Switch_THT:SW_PUSH_6mm, symbol Switch:SW_Push

Commit message: feat: fiducials, net classes, and a BAT sense divider
Fiducials (1 mm dot / 2 mm mask), three per populated face at three of the
four corners - never four, since a symmetric set gives the placement machine
no way to distinguish a 180-degree-rotated panel. Main board gets both faces
(FID1-3 front, FID4-6 back); the optical head is single-sided so its back has
none.

Net classes set in both .kicad_pro, sized from IPC-2221 at 1 oz outer copper
and a 10 C rise (0.20 mm ~ 0.74 A, 0.50 ~ 1.45 A, 0.80 ~ 2.03 A):
  Default 0.20  Power 0.50  Switch 0.80 (main)  Emitter 0.80 (head)  USB pair
Switch clearance stays at 0.20 rather than 0.25: the TPS63031's WSON-10 puts
its own L1/L2 pads 0.20 mm from its thermal pad, so anything stricter fails
inside the package. The USB class exists for tuning and length matching but is
not an impedance solution - that needs the fab's stackup. The S3's native USB
is Full Speed, so it matters less than it would at High Speed.

BAT sense divider - R33/R34 (1M) and C31 (100n) on GPIO4 (ADC1_CH3):
SUPPLY_SENSE reads SYS_SW/2 and cannot separate USB from battery, because a
USB port at the low end of spec minus D2's drop lands near 4.30 V against a
full cell at 4.20 V - inside divider tolerance plus ADC error. Comparing
SYS_SW against BAT is a differential test and separates them cleanly. 1M/1M
rather than 100k/100k because this divider hangs on the cell even when the
puck is off (~2 uA vs ~21 uA); the resulting 500k source impedance means
firmware needs a long sample time and multisample.

U1 pin 8's no-connect removed and U1.8 dropped from unused-pins.json.

verify_netlist.py spec extended with BAT_SENSE and the new ground/BAT members.
  main PASS: 44 exact circuit nets, 286 pin endpoints, 128 IC pads
  head PASS: 16 exact circuit nets, 63 pin endpoints
ERC 0 errors. DRC: main 2 (U1 library courtyard vs the corner holes), head 0.
All 81 schematic parts confirmed present on the board; the only board-only
refs are the 6 fiducials and 4 mounting hole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
Parts:
- added C31: 100n, Capacitor_SMD:C_0805_2012Metric, symbol Device:C
- added R33, R34: 1M, Resistor_SMD:R_0603_1608Metric, symbol Device:R
Connections:
- net BAT: now also R33.1
- net GND: now also C31.2, R34.2
- net BAT_SENSE: now reaches U1.8 (IO4)
- net BAT_SENSE: now also C31.1, R33.2, R34.1
- no-connect marks 36 -> 35
