File: BalancerREF/BalancerREF.kicad_sch (KiCad schematic)
At the start: 79 parts, among them J1 USB4105-GF-A, J2 LiPo 500mAh PROTECTED, J3 MAG+ / MAG- PTH, J4 GPS MODULE 3V3 UART, J5 OPTICAL HEAD 7-WAY, Q4 AO3401A, SW1 POWER, SW2 ACQUIRE, SW3 BOOT / SERVICE, U1 ESP32-S3-MINI-1-N8, U10 SN74LVC1G123DCTR, U2 IIS3DWBTR, U3 LM1815MX/NOPB, U5 BQ24075RGT, U6 TPS63031DSKR, U7 SRV05-4MR6T1G, U9 SN74LVC1G132DBVR

Commit message: feat: BalancerREF regrouped placement, hand routing, neck-down rules
Board: power chain regrouped into the top-right corner (U5 beside J2, U6
below it, SW1 on the right edge), USB channel cleared between J1 and U1,
passives re-clustered under their ICs. Seven test points dropped
(TP4/5/6/11/12/13/14). First pass of hand routing.

Rules: BalancerREF.kicad_dru necks Power-class tracks down to 0.2 mm and
vias to 0.5/0.3 inside the 0.5 mm pitch packages (U5, U6, U2, U10) and
0.3 mm in the SOT-23s (U7, U9).

Scripts: regroup_blocks.py (the placement pass, dry run by default) and
recover_from_dsn.py, which replays a Freerouting DSN export back onto the
saved board - used to recover the 22:00 session after the editor crashed
on session import.

Co-Authored-By: Claude Fable 5.1 <noreply@anthropic.com>
Parts:
- removed TP11: TP_USB_D+, TestPoint:TestPoint_Pad_D1.0mm, symbol Connector:TestPoint
- removed TP12: TP_USB_D-, TestPoint:TestPoint_Pad_D1.0mm, symbol Connector:TestPoint
- removed TP13: TP_EN, TestPoint:TestPoint_Pad_D1.0mm, symbol Connector:TestPoint
- removed TP14: TP_BOOT, TestPoint:TestPoint_Pad_D1.0mm, symbol Connector:TestPoint
- removed TP4: TP_USB_VBUS, TestPoint:TestPoint_Pad_D1.0mm, symbol Connector:TestPoint
- removed TP5: TP_MAG+, TestPoint:TestPoint_Pad_D1.0mm, symbol Connector:TestPoint
- removed TP6: TP_MAG-, TestPoint:TestPoint_Pad_D1.0mm, symbol Connector:TestPoint
Other:
- moved on the sheet: C1, C13, C14, C15, C16, C17, C18, C19, C2, C26, C27, C28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

Commit message: fix: BOM fields, silkscreen labels, +3V3 plane, and stale docs before review
- MPN fields: R3/R35/R36 (were "100k"), U9 (was the 1G08), R18 (was 3R0)
- Title block: HOBOVibe spelling; head company line no longer says "human
  review required"
- C20 on the head board rated 10 V; SYS_SW can sit at 5.5 V
- Silkscreen: board name and rev on both boards, battery and MAG polarity,
  pin-1 marks on J4 and both J5
- Main PCB: SYS, SYS_SW, BAT and USB_VBUS tracks removed from In2.Cu so the
  +3V3 plane is whole; three vias that only served them removed. Those four
  nets need re-routing on the outer layers.
- Docs: routing state, ground-pour wording, missing head-board holes,
  JLCPCB parts table rebuilt for the Rev F BOM, superseded LIS2DW12 and
  phototransistor sections marked in DATASHEET-VERIFICATION

Not done here (no KiCad in this environment): re-export of PDF/netlist/ERC/DRC.

Co-Authored-By: Claude Fable 5.1 <noreply@anthropic.com>
Claude-Session: https://claude.ai/code/session_01JeUyuyqf13Zf6V8TjfofPH
Parts:
- R3: MPN 100k -> 3.57k 1%
- R35: MPN 100k -> 1.6k
- R36: MPN 100k -> 10k
- U9: MPN SN74LVC1G08DBVR -> SN74LVC1G132DBVR
Other:
- title: HoboVibe Hobby Helicopter Dynamic Balancer -> HOBOVibe Hobby Helicopter Dynamic Balancer
Changed lines of the file:
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@@
 	(paper "A2")
 	(title_block
-		(title "HoboVibe Hobby Helicopter Dynamic Balancer")
+		(title "HOBOVibe Hobby Helicopter Dynamic Balancer")
 		(date "2026-09-13")
 		(rev "F")
@@
 			)
 		)
-		(property "MPN" "100k"
+		(property "MPN" "10k"
 			(at 254 140.97 0)
 			(hide yes)
@@
 			)
 		)
-		(property "MPN" "100k"
+		(property "MPN" "1.6k"
 			(at 234.95 140.97 0)
 			(hide yes)
@@
 			)
 		)
-		(property "MPN" "SN74LVC1G08DBVR"
+		(property "MPN" "SN74LVC1G132DBVR"
 			(at 149.86 285.75 0)
 			(hide yes)
@@
 			)
 		)
-		(property "MPN" "100k"
+		(property "MPN" "3.57k 1%"
 			(at 214.63 140.97 0)
 			(hide yes)

Commit message: fix: Rev G - D3 polarity, USB lines through U7, U9 pull-down, sharper review images
Three corrections from the Reddit review of the Rev C sheet, all still present in
Rev F:

- D3 (SMF5.0A, unidirectional TVS on USB_VBUS) was drawn cathode to GND and anode
  to VBUS: forward biased across the port. Cathode (pin 1) now on USB_VBUS; the
  D_SMF footprint is rotated 180 so pad 1 lands on the VBUS copper.
  DATASHEET-VERIFICATION had recorded the part as bidirectional; corrected.
- U7 (SRV05-4) pins 4 and 6 were NC and D+/D- hung off the array as stubs. The
  drawing now takes D- in at pin 1 and out at pin 6, D+ in at pin 3 and out at
  pin 4 (the opposite pads of the SOT-23-6). Nets stay the same on both sides,
  since the SRV05-4 has no internal I/O path: the trace has to join the pads.
  Board pads 4/6 carry the nets; the USB data routing itself is still to do.
- U9 pin 1 (OPT_COMP) floats when the optical head is unplugged, the normal
  state in MR-VERT. R39 100k to GND added, placed on the back under U9, unrouted.

Review outputs regenerated with kicad-cli 10.0.6: netlist, ERC, pin CSVs,
manifest, DRC report, schematic PDF. review/reddit/ re-rendered from Rev G at
400 DPI (full sheet) and 600 DPI (blocks); the old set was Rev C at ~216 DPI.
verify_netlist.py updated for the new nets and for TP4/5/6/11-14, which
58b622f had dropped from the sheet without updating the expected circuits.

Scripts: rev_g_usb_esd_tvs_u9.py (schematic), sync_board_rev_g.py (board),
render_review_images.py (images).

Co-Authored-By: Claude Fable 5.1 <noreply@anthropic.com>
Claude-Session: https://claude.ai/code/session_01RAWf9Skey6ZcU82AJn2CyR
Parts:
- added R39: 100k, Resistor_SMD:R_0603_1608Metric, symbol Device:R
Connections:
- net GND: now also D3.2 (A2), R39.1; no longer D3.1 (A1)
- net OPT_COMP: now also R39.2
- net USB_CONN_D+: now also U7.4 (IO3)
- net USB_CONN_D-: now also U7.6 (IO4)
- net USB_VBUS: now also D3.1 (A1); no longer D3.2 (A2)
- no-connect marks 32 -> 30
Other:
- note added: "U7: route each data line THROUGH the array. D- enters pin 1 and leaves pin 6, D+ enters pin 3 and leaves pin 4; the opposite pads sit across from each other."
- moved on the sheet: C1, D3
