File: BalancerREF/BalancerREF.kicad_pcb (KiCad board)
At the start: 4 copper layers, 50 x 50 mm, 79 parts, among them J1 USB4105-GF-A, J2 LiPo 500mAh PROTECTED, J3 MAG+ / MAG- PTH, J4 GPS MODULE 3V3 UART, J5 OPTICAL HEAD 7-WAY, Q4 AO3401A, SW1 POWER, SW2 ACQUIRE, SW3 BOOT / SERVICE, U1 ESP32-S3-MINI-1-N8, U10 SN74LVC1G123DCTR, U2 IIS3DWBTR, U3 LM1815MX/NOPB, U5 BQ24075RGT, U6 TPS63031DSKR, U7 SRV05-4MR6T1G, U9 SN74LVC1G132DBVR

Commit message: fix: Rev G - D3 polarity, USB lines through U7, U9 pull-down, sharper review images
Three corrections from the Reddit review of the Rev C sheet, all still present in
Rev F:

- D3 (SMF5.0A, unidirectional TVS on USB_VBUS) was drawn cathode to GND and anode
  to VBUS: forward biased across the port. Cathode (pin 1) now on USB_VBUS; the
  D_SMF footprint is rotated 180 so pad 1 lands on the VBUS copper.
  DATASHEET-VERIFICATION had recorded the part as bidirectional; corrected.
- U7 (SRV05-4) pins 4 and 6 were NC and D+/D- hung off the array as stubs. The
  drawing now takes D- in at pin 1 and out at pin 6, D+ in at pin 3 and out at
  pin 4 (the opposite pads of the SOT-23-6). Nets stay the same on both sides,
  since the SRV05-4 has no internal I/O path: the trace has to join the pads.
  Board pads 4/6 carry the nets; the USB data routing itself is still to do.
- U9 pin 1 (OPT_COMP) floats when the optical head is unplugged, the normal
  state in MR-VERT. R39 100k to GND added, placed on the back under U9, unrouted.

Review outputs regenerated with kicad-cli 10.0.6: netlist, ERC, pin CSVs,
manifest, DRC report, schematic PDF. review/reddit/ re-rendered from Rev G at
400 DPI (full sheet) and 600 DPI (blocks); the old set was Rev C at ~216 DPI.
verify_netlist.py updated for the new nets and for TP4/5/6/11-14, which
58b622f had dropped from the sheet without updating the expected circuits.

Scripts: rev_g_usb_esd_tvs_u9.py (schematic), sync_board_rev_g.py (board),
render_review_images.py (images).

Co-Authored-By: Claude Fable 5.1 <noreply@anthropic.com>
Claude-Session: https://claude.ai/code/session_01RAWf9Skey6ZcU82AJn2CyR
Parts:
- added R39: 100k, R_0603_1608Metric, B.Cu at (113.8, 115.2)
- turned D3 to 0 degrees
Connections:
- D3 pad 1: GND -> /USB_VBUS
- D3 pad 2: /USB_VBUS -> GND
- U7 pad 4: unconnected-(U7-IO3-Pad4) -> /USB_CONN_D+
- U7 pad 6: unconnected-(U7-IO4-Pad6) -> /USB_CONN_D-
Other:
- board text added: "HOBOVibe RevG"
- board text removed: "HOBOVibe RevF"
