File: BalancerREF_OptHead/BalancerREF_OptHead.kicad_sch (KiCad schematic)
At the start: 24 parts, among them J5 TO MAIN BOARD, Q1 AO3400A, U4 TS3021IYLT, U8 TLV9062IDR

Commit message: fix: address repo review findings before routing
An external review raised seven pre-routing items plus smaller notes. Each was
checked against the manufacturer source rather than taken on faith; two did not
survive that check and are recorded as not-confirmed.

Confirmed and fixed:

  * D1 peak current. The head runs from SYS_SW, and with the BQ24075 regulating
    OUT to 5.5 V, R18 at 3.0 ohm gave ~1.1 A peak against D1's 1 A absolute
    maximum. The BOM note had only checked the 4.2 V battery case, and the
    charger swap - which replaced a Schottky holding SYS near 4.55 V - is what
    pushed it over. R18 -> 3.9 ohm: ~0.49 A at a full cell (the bench-set design
    point) and ~0.90 A worst case at 5.5 V with a low-Vf bin.
  * Charger stuck at USB100. EN1/EN2 have 285k internal pulldowns and nothing
    drove them, so the input limit covered system load AND charge current at
    100 mA. setupCharger() now selects USB500 at boot, and status reports
    input_present/charging from PGOOD and CHG.
  * U9 input transition rate. R29/C26 fed the SN74LVC1G08 a 0.47 us edge against
    a 10 ns/V spec, ~25x out. Swapped to SN74LVC1G132, a Schmitt NAND with the
    identical SOT-23-5 pinout (verified against SLVS322 Figure 4-1), which
    conditions both inputs. It inverts, so U10's trigger moved from B rising to
    ~A falling - the SN74LVC1G123 supports both edges.
  * Switcher parts on the wrong face. L1 and C4-C7 were on the back with U6 on
    the front, putting vias in a 2.4 MHz switching loop. Moved to the front;
    C2/C3/C30 followed for the BQ24075. The "ICs front, passives back" rule does
    not survive contact with a switching converter.
  * U1 decoupling. C8 is now 0.38 mm from the 3V3 pad instead of ~9 mm. Both
    stay on the back, since U1's body owns that part of the front.
  * Head board emitter loop, was spanning the full board width. C20/R18/Q1 now
    cluster in 6.9 x 3.3 mm. R21/C21 went from 4 mm off Q1 to 16 mm and sit
    3.6/3.9 mm from U8 pins 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
Parts:
- R18: value 3R0 1206 0.5W -> 3R9 1206 0.5W
