File: BalancerREF_OptHead/BalancerREF_OptHead.kicad_sch (KiCad schematic)
At the start: 28 parts, among them J5 TO MAIN BOARD, Q1 AO3400A, U4 TS3021IYLT, U8 TLV9062IDR

Commit message: feat: carrier J5 moved toward the optical head; head gain redistributed
Carrier: J5 moved up the left edge, next to the optical head, clear of the
FeatherS3[D] battery connector, opening away from the module. Each J5 ground
pin and 3V3 now drops to its plane through its own via within ~2 mm, and
OPT_COMP no longer runs alongside OPT_LED_EN. DRC 0 violations, 0
unconnected, 0 schematic parity (with the local U5 LGA pad-to-pad rule).

Optical head: R21 10k -> 4.99k, R23 120k -> 240k, C21 22p -> 47p C0G. Same
~120 kOhm total gain with about twice the TIA ambient headroom (~160 to
~320 uA photocurrent), per the 2026-09-23 SPICE review; to be bench-tested
before production. Silkscreen cleanup clears the previous DRC warnings.
DRC 0 violations, 0 unconnected; the 3 parity items are mounting holes and
fiducials without symbols.

Co-Authored-By: Claude Opus 5.5 <noreply@anthropic.com>
Parts:
- C21: value 22p C0G -> 47p C0G; MPN 22p C0G -> 47p C0G
- R21: value 10k -> 4.99k; MPN 10k -> 4.99k
- R23: value 120k -> 240k; MPN 120k -> 240k
Changed lines of the file:
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@@
 			)
 		)
-		(property "Value" "10k"
+		(property "Value" "4.99k"
 			(at 165.1 78.74 90)
 			(show_name no)
@@
 			)
 		)
-		(property "MPN" "10k"
+		(property "MPN" "4.99k"
 			(at 165.1 73.66 90)
 			(hide yes)
@@
 			)
 		)
-		(property "Value" "22p C0G"
+		(property "Value" "47p C0G"
 			(at 165.1 62.23 90)
 			(show_name no)
@@
 			)
 		)
-		(property "MPN" "22p C0G"
+		(property "MPN" "47p C0G"
 			(at 165.1 63.5 90)
 			(hide yes)
@@
 			)
 		)
-		(property "Value" "120k"
+		(property "Value" "240k"
 			(at 248.92 81.28 90)
 			(show_name no)
@@
 			)
 		)
-		(property "MPN" "120k"
+		(property "MPN" "240k"
 			(at 248.92 76.2 90)
 			(hide yes)
