File: BalancerCarrier/BalancerCarrier.kicad_sch (KiCad schematic)
At the start: 31 parts, among them J3 MAG+ / MAG- PTH, J4 GPS MODULE 3V3 UART, J5 OPTICAL HEAD 7-WAY, SW1 ACQUIRE, U1 FeatherS3[D], U2 LM1815MX/NOPB, U3 SN74LVC1G132DBVR, U4 SN74LVC1G123DCTR, U5 IIS3DWBTR

Commit message: feat: carrier PCB first layout, schematic fixes, OptHead 3D models
BalancerCarrier
  - First .kicad_pcb into git: 4 layers, 139 tracks, 51 vias, GND on In1.Cu
    and +3V3 on In2.Cu, 0 unconnected. Placement recovered from
    temp-freerouting.dsn after the Freerouting crash took the board file.
  - Schematic fixes found in review: LED1 was wired backwards (cathode on the
    GPIO), R13 sat in series with J5.5 instead of returning to GND, and
    GPS_UART_RX collided with the module I2C bus on IO9 - moved to IO7.
  - The GPS block is kept but DNP for the first round; the board is a
    proof-of-concept that the balancer works before the GPS is added on.
  - .kicad_pro carries the netclasses the board's DRC depends on, so it goes
    in with the board rather than after it.
  - scripts/restore_placement_pcbnew.py is the recovery tool that worked.
    restore_placement_from_dsn.py is kept beside it with a header explaining
    why editing the file directly shears the pads: KiCad stores each pad's
    angle including its parent footprint's.

BalancerREF_OptHead
  - PD1 is now an SFH 2440. The SFH 2430 it replaces has a 200 us rise time
    against the 2440's 0.09 us, which cannot resolve a rotor blade passing.
  - 3D models attached to D1 and PD1.

Known, not fixed here: 13 DRC violations on the carrier, 12 of them U5's LGA
pad-to-pad gap of 0.150 mm against the 0.2 mm netclass clearance (needs a
local override, not a layout change), and one benign J3 THT layer mismatch.
Parts:
- added H1, H2, H3, H4, H5: MountingHole, MountingHole:MountingHole_2.2mm_M2, symbol Mechanical:MountingHole
Connections:
- net VR_IN: no longer names the net of R6.2, U2.3 (VR_IN)
Other:
- moved on the sheet: C11, C12, C2, C3, C4, C5, C6, C7, C8, C9, J3, J4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
