File: BalancerCarrier/BalancerCarrier.kicad_sch (KiCad schematic)
At the start: 36 parts, among them J3 MAG+ / MAG- PTH, J4 GPS MODULE 3V3 UART, J5 OPTICAL HEAD 7-WAY, SW1 ACQUIRE, U1 FeatherS3[D], U2 LM1815MX/NOPB, U3 SN74LVC1G132DBVR, U4 SN74LVC1G123DCTR, U5 IIS3DWBTR

Commit message: feat: carrier J5 moved toward the optical head; head gain redistributed
Carrier: J5 moved up the left edge, next to the optical head, clear of the
FeatherS3[D] battery connector, opening away from the module. Each J5 ground
pin and 3V3 now drops to its plane through its own via within ~2 mm, and
OPT_COMP no longer runs alongside OPT_LED_EN. DRC 0 violations, 0
unconnected, 0 schematic parity (with the local U5 LGA pad-to-pad rule).

Optical head: R21 10k -> 4.99k, R23 120k -> 240k, C21 22p -> 47p C0G. Same
~120 kOhm total gain with about twice the TIA ambient headroom (~160 to
~320 uA photocurrent), per the 2026-09-23 SPICE review; to be bench-tested
before production. Silkscreen cleanup clears the previous DRC warnings.
DRC 0 violations, 0 unconnected; the 3 parity items are mounting holes and
fiducials without symbols.

Co-Authored-By: Claude Opus 5.5 <noreply@anthropic.com>
Parts:
- added C14: 100n, Capacitor_SMD:C_0805_2012Metric, symbol Device:C
- J3: now left out of the parts list
Connections:
- net +3V3: now also C14.1
- net GND: now also C14.2
Changed lines of the file:
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@@
 	)
 	(symbol
+		(lib_id "power:+3V3")
+		(at 288.925 160.655 0)
+		(unit 1)
+		(body_style 1)
+		(exclude_from_sim no)
+		(in_bom yes)
+		(on_board yes)
+		(in_pos_files yes)
+		(dnp no)
+		(fields_autoplaced yes)
+		(property "Reference" "#PWR020"
+			(at 288.925 164.465 0)
+			(hide yes)
+			(show_name no)
+			(do_not_autoplace no)
+			(effects
+				(font
+					(size 1.27 1.27)
+				)
+			)
+		)
+		(property "Value" "+3V3"
+			(at 288.925 156.21 0)
+			(show_name no)
+			(do_not_autoplace no)
+			(effects
+				(font
+					(size 1.27 1.27)
+				)
+			)
+		)
+		(property "Footprint" ""
+			(at 288.925 160.655 0)
+			(hide yes)
+			(show_name no)
+			(do_not_autoplace no)
+			(effects
+				(font
+					(size 1.27 1.27)
+				)
+			)
+		)
+		(property "Datasheet" ""
+			(at 288.925 160.655 0)
+			(hide yes)
+			(show_name no)
+			(do_not_autoplace no)
+			(effects
+				(font
+					(size 1.27 1.27)
+				)
+			)
+		)
+		(property "Description" "Power symbol creates a global label with name \"+3V3\""
+			(at 288.925 160.655 0)
+			(hide yes)
+			(show_name no)
+			(do_not_autoplace no)
+			(effects
+				(font
+					(size 1.27 1.27)
+				)
+			)
+		)
+		(pin "1"
+		)
+		(instances
+			(project "BalancerCarrier"
+				(path "/b1c0a5d2-0e41-4a7f-9d3c-1f2e3a4b5c6d"
+					(reference "#PWR020")
+					(unit 1)
+				)
+			)
+		)
+	)
+	(symbol
 		(lib_id "Device:LED")
 		(at 292.1 137.16 180)
@@
 		(body_style 1)
 		(exclude_from_sim no)
-		(in_bom yes)
+		(in_bom no)
 		(on_board yes)
 		(in_pos_files yes)
@@
 					(unit 1)
 				)
+			)
+		)
+	)
+	(symbol
+		(lib_id "Device:C")
+		(at 288.925 164.465 0)
+		(unit 1)
+		(body_style 1)
+		(exclude_from_sim no)
+		(in_bom yes)
+		(on_board yes)
+		(in_pos_files yes)
+		(dnp no)
+		(fields_autoplaced yes)
+		(property "Reference" "C14"
+			(at 292.1 163.1949 0)
+			(show_name no)
+			(do_not_autoplace no)
+			(effects
+				(font
+					(size 1.27 1.27)
+				)
+				(justify left)
+			)
+		)
+		(property "Value" "100n"
+			(at 292.1 165.7349 0)
+			(show_name no)
+			(do_not_autoplace no)
+			(effects
+				(font
+					(size 1.27 1.27)
+				)
+				(justify left)
+			)
+		)
+		(property "Footprint" "Capacitor_SMD:C_0805_2012Metric"
+			(at 289.8902 168.275 0)
+			(hide yes)
+			(show_name no)
+			(do_not_autoplace no)
+			(effects
+				(font
+					(size 1.27 1.27)
+				)
+			)
+		)
+		(property "Datasheet" ""
+			(at 288.925 164.465 0)
+			(hide yes)
+			(show_name no)
+			(do_not_autoplace no)
+			(effects
+				(font
+					(size 1.27 1.27)
+				)
+			)
+		)
+		(property "Description" "Unpolarized capacitor"
+			(at 288.925 164.465 0)
+			(hide yes)
+			(show_name no)
+			(do_not_autoplace no)
+			(effects
+				(font
+					(size 1.27 1.27)
+				)
+			)
+		)
+		(pin "2"
+		)
+		(pin "1"
+		)
+		(instances
+			(project "BalancerCarrier"
+				(path "/b1c0a5d2-0e41-4a7f-9d3c-1f2e3a4b5c6d"
+					(reference "C14")
+					(unit 1)
+				)
+			)
+		)
+	)
+	(symbol
+		(lib_id "power:GND")
+		(at 288.925 168.275 0)
+		(unit 1)
+		(body_style 1)
+		(exclude_from_sim no)
+		(in_bom yes)
+		(on_board yes)
+		(in_pos_files yes)
+		(dnp no)
+		(fields_autoplaced yes)
+		(property "Reference" "#PWR021"
+			(at 288.925 174.625 0)
+			(hide yes)
+			(show_name no)
+			(do_not_autoplace no)
+			(effects
+				(font
+					(size 1.27 1.27)
+				)
+			)
+		)
+		(property "Value" "GND"
+			(at 288.925 172.72 0)
+			(show_name no)
+			(do_not_autoplace no)
+			(effects
+				(font
+					(size 1.27 1.27)
+				)
+			)
+		)
+		(property "Footprint" ""
+			(at 288.925 168.275 0)
+			(hide yes)
+			(show_name no)
+			(do_not_autoplace no)
+			(effects
+				(font
+					(size 1.27 1.27)
+				)
+			)
+		)
+		(property "Datasheet" ""
+			(at 288.925 168.275 0)
+			(hide yes)
+			(show_name no)
+			(do_not_autoplace no)
+			(effects
+				(font
+					(size 1.27 1.27)
+				)
+			)
+		)
+		(property "Description" "Power symbol creates a global label with name \"GND\" , ground"
+			(at 288.925 168.275 0)
+			(hide yes)
+			(show_name no)
+			(do_not_autoplace no)
+			(effects
+				(font
+					(size 1.27 1.27)
+				)
+			)
+		)
+		(pin "1"
+		)
+		(instances
+			(project "BalancerCarrier"
+				(path "/b1c0a5d2-0e41-4a7f-9d3c-1f2e3a4b5c6d"
+					(reference "#PWR021")
+					(unit 1)
+				)
